File: IO4-IR-Detector-Active-Fingers.sch (EAGLE design)
At the start: 32 parts, among them J1 0.100, J10 0.100, J11 0.100, J12 0.100, J13 0.100, J14 0.100, J15 0.100, J16 0.100, J2 0.100, J3 0.100, J4 0.100, J5 0.100, J6 0.100, J7 0.100, J8 0.100, J9 0.100, U1 QRE1113, U10 QRE1113, U11 QRE1113, U12 QRE1113, U13 QRE1113, U14 QRE1113, U15 QRE1113, U16 QRE1113, U2 QRE1113, U3 QRE1113, U4 QRE1113, U5 QRE1113, U6 QRE1113, U7 QRE1113, U8 QRE1113, U9 QRE1113

Commit message: silk
Other:
- note added: "1.3"
- note added: "HO"
- note removed: "1.0"
- note removed: "A"
Changed lines of the file:
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@@
 <plain>
 <text x="151.13" y="19.558" size="2.54" layer="91">Reflected IR Light detector</text>
-<text x="241.3" y="12.7" size="2.54" layer="91">1.0</text>
-<text x="241.808" y="6.096" size="2.54" layer="91">A</text>
+<text x="241.3" y="12.7" size="2.54" layer="91">1.3</text>
+<text x="241.808" y="6.096" size="2.54" layer="91">HO</text>
 </plain>
 <instances>
